Commit message: changed

File: src/srobot_gazebo/urdf/srobot.gazebo.xacro (robot description, xacro)
@@ -36,19 +36,20 @@
     <material>Gazebo/FlatBlack</material>
   </gazebo>
-  <gazebo reference="imu">
+ <gazebo reference="imu_link">
     <gravity>true</gravity>
     <sensor name="imu_sensor" type="imu">
       <always_on>true</always_on>
       <update_rate>100</update_rate>
-      <visualize>true</visualize>
+      <visualize>false</visualize>
       <topic>__default_topic__</topic>
       <plugin filename="libgazebo_ros_imu_sensor.so" name="imu_plugin">
         <topicName>imu</topicName>
-        <bodyName>imu</bodyName>
+        <bodyName>imu_link</bodyName>
         <updateRateHZ>10.0</updateRateHZ>
         <gaussianNoise>0.0</gaussianNoise>
         <xyzOffset>0 0 0</xyzOffset>
         <rpyOffset>0 0 0</rpyOffset>
-        <frameName>imu</frameName>
+        <frameName>imu_link</frameName>
+        <initialOrientationAsReference>false</initialOrientationAsReference>
       </plugin>
       <pose>0 0 0 0 0 0</pose>
@@ -61,9 +62,9 @@
       <odometryFrame>odom</odometryFrame>
       <odometrySource>world</odometrySource>
-      <publishOdomTF>true</publishOdomTF>
+      <publishOdomTF>flase</publishOdomTF>
       <robotBaseFrame>base_footprint</robotBaseFrame>
       <publishWheelTF>false</publishWheelTF>
-      <publishTf>true</publishTf>
-      <publishWheelJointState>true</publishWheelJointState>
+      <publishTf>flase</publishTf>
+      <publishWheelJointState>false</publishWheelJointState>
       <legacyMode>false</legacyMode>
       <updateRate>30</updateRate>

File: src/srobot_gazebo/urdf/srobot.xacro (robot description, xacro)
@@ -112,5 +112,5 @@
   </joint>
   <!-- imu sensor -->
-  <link name="imu">
+  <link name="imu_link">
     <visual>
       <geometry>
@@ -124,5 +124,5 @@
   <joint name="imu_joint" type="fixed">
     <parent link="base_footprint"/>
-    <child link="imu"/>
+    <child link="imu_link"/>
     <origin xyz="0.08 0 0.025"/>
   </joint>
